Commit message: Variable length world bouds. Units adapted to metres.

File: spike_swarm_sim/objects/urdf/wall.urdf (robot description, URDF)
Before this commit: robot wall, 1 links, 0 joints
Links:
- link baseLink: geometry collision box size=1 11 2; visual box size=1 11 2

Commit message: Distance sensor and obs. avoidance fitness slightly changed.

File: spike_swarm_sim/objects/urdf/wall.urdf (robot description, URDF)
Before this commit: robot wall, 1 links, 0 joints
Links:
- link baseLink: geometry collision box size=1 8 2; visual box size=1 8 2
