Commit message: New epuck model. 3D distance sensor bug fixed.

File: spike_swarm_sim/objects/urdf/epuck.urdf (robot description, URDF)
Before this commit: robot epuck, 6 links, 5 joints
Links:
- removed link LED
- removed link aux_wheel
- removed link aux_wheel2
- added link cam, mass 0.005; collision mesh filename=cam.obj scale=0.5 0.5 0.5; visual mesh filename=cam.obj scale=0.5 0.5 0.5
- added link leds, mass 0.01; collision mesh filename=led_base.obj scale=0.5 0.5 0.5; visual mesh filename=led_base.obj scale=0.5 0.5 0.5
- added link top, mass 0.01; collision mesh filename=epuck_top.obj scale=0.5 0.5 0.5; visual mesh filename=epuck_top.obj scale=0.5 0.5 0.5
- link base_link: mass 2 -> 1; geometry collision mesh filename=epuck_body.obj scale=0.5 0.5 0.5; visual mesh filename=epuck_body.obj scale=0.5 0.5 0.5
- link left_wheel: mass 0.2 -> 0.01; geometry collision mesh filename=wheel.obj scale=0.5 0.25 0.5; visual mesh filename=wheel.obj scale=0.5 0.25 0.5
- link right_wheel: mass 0.2 -> 0.01; geometry collision mesh filename=wheel.obj scale=0.5 0.25 0.5; visual mesh filename=wheel.obj scale=0.5 0.25 0.5
Joints:
- removed joint base_to_LED
- removed joint base_to_aux_wheel
- removed joint base_to_aux_wheel2
- added joint base_to_cam: type fixed, parent base_link, child cam, origin xyz=0.268 0.0 0.07 rpy=3.1415 1.57075 0
- added joint base_to_leds: type fixed, parent base_link, child leds, origin xyz=0 -0.098 0.12 rpy=1.57075 0 0
- added joint base_to_top: type fixed, parent base_link, child top, origin xyz=0 -0.098 0.12 rpy=1.57075 0 0
- joint base_to_left_wheel: axis 0 0 1 -> 0 1 0; origin xyz=0 0.109 -0.01 rpy=1.57075 0 0 -> xyz=0.007 0.12 0.078 rpy=0 0 0
- joint base_to_right_wheel: axis 0 0 1 -> 0 1 0; origin xyz=0.0 -0.109 -0.01 rpy=1.57075 0 0 -> xyz=0.007 -0.12 0.078 rpy=0 0 0

File: spike_swarm_sim/objects/urdf/wall.urdf (robot description, URDF)
Before this commit: robot wall, 1 links, 0 joints
Links:
- link baseLink: mass 100.0 -> 1000.0

Commit message: Bug zero mass of links in linux detected and fixed provisionally.

File: spike_swarm_sim/objects/urdf/epuck.urdf (robot description, URDF)
Before this commit: robot epuck, 6 links, 5 joints
Links:
- link left_wheel: mass 0.01 -> 0.05
- link right_wheel: mass 0.01 -> 0.05

Commit message: Bug zero mass of links in linux detected and fixed provisionally.

File: spike_swarm_sim/objects/urdf/epuck.urdf (robot description, URDF)
Before this commit: robot epuck, 6 links, 5 joints
Links:
- link base_link: mass 1 -> 3
- link cam: mass 0.005 -> 0.0
- link leds: mass 0.01 -> 1
- link left_wheel: mass 0.05 -> 1
- link right_wheel: mass 0.05 -> 1

Commit message: Minor changes.

File: spike_swarm_sim/objects/urdf/epuck.urdf (robot description, URDF)
Before this commit: robot epuck, 6 links, 5 joints
Links:
- link base_link: mass 3 -> 1
- link top: mass 0.01 -> 0.0

Commit message: IR sensors added to URDF. Distance sensor 3D updated.

File: spike_swarm_sim/objects/urdf/epuck.urdf (robot description, URDF)
Before this commit: robot epuck, 6 links, 5 joints
Links:
- added link IR0, mass 0.0; collision mesh filename=ir.obj scale=1 1 1; visual mesh filename=ir.obj scale=1 1 1
- added link IR1, mass 0.0; collision mesh filename=ir.obj scale=1 1 1; visual mesh filename=ir.obj scale=1 1 1
- added link IR2, mass 0.0; collision mesh filename=ir.obj scale=1 1 1; visual mesh filename=ir.obj scale=1 1 1
- added link IR3, mass 0.0; collision mesh filename=ir.obj scale=1 1 1; visual mesh filename=ir.obj scale=1 1 1
- added link IR4, mass 0.0; collision mesh filename=ir.obj scale=1 1 1; visual mesh filename=ir.obj scale=1 1 1
- added link IR5, mass 0.0; collision mesh filename=ir.obj scale=1 1 1; visual mesh filename=ir.obj scale=1 1 1
- link base_link: mass 0.1 -> 1
- link cam: mass 0.0 -> 0.005
- link top: mass 0.0 -> 0.01
Joints:
- added joint base_to_IR0: type fixed, parent base_link, child IR0, origin xyz=0.16 0.0 0.127 rpy=1.2 0 1.5707963267948966
- added joint base_to_IR1: type fixed, parent base_link, child IR1, origin xyz=0.08000000000000002 0.13856406460551018 0.127 rpy=1.2 0 2.617993877991494
- added joint base_to_IR2: type fixed, parent base_link, child IR2, origin xyz=-0.07999999999999996 0.13856406460551018 0.127 rpy=1.2 0 3.665191429188092
- added joint base_to_IR3: type fixed, parent base_link, child IR3, origin xyz=-0.16 1.959434878635765e-17 0.127 rpy=1.2 0 4.71238898038469
- added joint base_to_IR4: type fixed, parent base_link, child IR4, origin xyz=-0.08000000000000007 -0.13856406460551016 0.127 rpy=1.2 0 5.759586531581287
- added joint base_to_IR5: type fixed, parent base_link, child IR5, origin xyz=0.07999999999999989 -0.13856406460551024 0.127 rpy=1.2 0 6.8067840827778845

Commit message: Fixed problem of multiproc. unstab. (still happens with insignificantly). Side walls variable dimensions updated.

File: spike_swarm_sim/objects/urdf/epuck.urdf (robot description, URDF)
Before this commit: robot epuck, 12 links, 11 joints
Links:
- link base_link: mass 1 -> 1.5
- link left_wheel: mass 0.01 -> 0.1
- link right_wheel: mass 0.01 -> 0.1
- link top: mass 0.01 -> 0.5

Commit message: Orientation arrow 3D added to Epuck urdf.

File: spike_swarm_sim/objects/urdf/epuck.urdf (robot description, URDF)
Before this commit: robot epuck, 12 links, 11 joints
Links:
- added link arrow, mass 0; collision mesh filename=arrow.obj scale=0.1 0.1 0.1; visual mesh filename=arrow.obj scale=0.1 0.1 0.1
Joints:
- added joint base_to_arrow: type fixed, parent base_link, child arrow, origin xyz=0 0.0 0.15 rpy=0 0 0

Commit message: Epuck 3D IR model improved. SNES init sigma slightly increased.

File: spike_swarm_sim/objects/urdf/epuck.urdf (robot description, URDF)
Before this commit: robot epuck, 13 links, 12 joints
Links:
- removed link IR4
- removed link IR5
Joints:
- removed joint base_to_IR4
- removed joint base_to_IR5
- joint base_to_IR1: origin xyz=0.08000000000000002 0.13856406460551018 0.127 rpy=1.2 0 2.617993877991494 -> xyz=9.797174393178826e-18 0.16 0.127 rpy=1.2 0 3.141592653589793
- joint base_to_IR2: origin xyz=-0.07999999999999996 0.13856406460551018 0.127 rpy=1.2 0 3.665191429188092 -> xyz=-0.16 1.959434878635765e-17 0.127 rpy=1.2 0 4.71238898038469
- joint base_to_IR3: origin xyz=-0.16 1.959434878635765e-17 0.127 rpy=1.2 0 4.71238898038469 -> xyz=-2.9391523179536474e-17 -0.16 0.127 rpy=1.2 0 6.283185307179586
