Commit message: Ground sensor and sectorized color sensor implemented. Cube transportation config file started.

File: spike_swarm_sim/objects/urdf/cube.urdf (robot description, URDF)
Before this commit: robot light, 1 links, 0 joints
Links:
- link baseLink: geometry collision mesh filename=cube.obj scale=1 1 1; visual mesh filename=cube.obj scale=1 1 1
