Commit message: Directional sensors revisited: using coverage cones and batch rays to detect obstacles and targets.

File: spike_swarm_sim/models/maps/complex_maze_1/complex_maze_1.urdf (robot description, URDF)
Before this commit: robot tmaze.urdf, 1 links, 0 joints
Links:
- link baseLink: geometry collision mesh filename=complex_maze_1.obj scale=3 1 3; visual mesh filename=complex_maze_1.obj scale=3 1 3

File: spike_swarm_sim/objects/urdf/wall.urdf (robot description, URDF)
Before this commit: robot wall, 1 links, 0 joints
Links:
- link baseLink: mass 1000.0 -> 0.0
