Commit message: Basic examples ready to go (not documented yet). Docs tutorials (worlds and entities) improved. Docs installation. Minor code changes.

File: spike_swarm_sim/models/entities/epuck/epuck.urdf (robot description, URDF)
Before this commit: robot epuck, 23 links, 22 joints
Links:
- removed link leds
- added link led0, mass 0.01; collision mesh filename=led0.obj scale=0.5 0.5 0.5; visual mesh filename=led0.obj scale=0.5 0.5 0.5
- link ghost_cone_DS0: geometry collision mesh filename=cone.obj scale=1 1 1; visual mesh filename=cone.obj scale=1 1 1
- link ghost_cone_DS1: geometry collision mesh filename=cone.obj scale=1 1 1; visual mesh filename=cone.obj scale=1 1 1
- link ghost_cone_DS2: geometry collision mesh filename=cone.obj scale=1 1 1; visual mesh filename=cone.obj scale=1 1 1
- link ghost_cone_DS3: geometry collision mesh filename=cone.obj scale=1 1 1; visual mesh filename=cone.obj scale=1 1 1
- link ghost_cone_DS4: geometry collision mesh filename=cone.obj scale=1 1 1; visual mesh filename=cone.obj scale=1 1 1
- link ghost_cone_DS5: geometry collision mesh filename=cone.obj scale=1 1 1; visual mesh filename=cone.obj scale=1 1 1
- link ghost_cone_DS6: geometry collision mesh filename=cone.obj scale=1 1 1; visual mesh filename=cone.obj scale=1 1 1
- link ghost_cone_DS7: geometry collision mesh filename=cone.obj scale=1 1 1; visual mesh filename=cone.obj scale=1 1 1
Joints:
- removed joint base_to_leds
- added joint base_to_led0: type fixed, parent base_link, child led0, origin xyz=0 -0.098 0.12 rpy=1.57075 0 0

File: spike_swarm_sim/models/entities/light_source/light.urdf (robot description, URDF)
Before this commit: robot light, 1 links, 0 joints
Links:
- link baseLink: geometry collision mesh filename=sphere.obj scale=0.4 0.4 0.4; visual mesh filename=sphere.obj scale=0.4 0.4 0.4
