Commit message: Debugging trace removed from basic example 2.

File: spike_swarm_sim/models/entities/epuck/epuck.urdf.xacro (robot description, xacro)
@@ -104,8 +104,8 @@
         <visual>
             <geometry>
-                <mesh filename="led_0.obj" scale="1.5 1.5 1.5" />
-            </geometry>
-            <origin xyz="0 0 0" />
-            <material name="white">
+                <mesh filename="led_0.obj" scale=".5 .5 .5" />
+            </geometry>
+            <origin xyz="0 0 0" />
+            <material name="transparent_white">
                 <color rgba="1 1 1 0.5" />
             </material>
@@ -113,5 +113,5 @@
         <collision>
             <geometry>
-               <mesh filename="led_0.obj" scale="1.5 1.5 1.5" />
+               <mesh filename="led_0.obj" scale=".5 .5 .5" />
             </geometry>
             <origin xyz="0 0 0" />
@@ -125,8 +125,8 @@
         <visual>
             <geometry>
-                <mesh filename="led_1.obj" scale="1.5 1.5 1.5" />
-            </geometry>
-            <origin xyz="0 0 0" />
-            <material name="white">
+                <mesh filename="led_1.obj" scale=".5 .5 .5" />
+            </geometry>
+            <origin xyz="0 0 0" />
+            <material name="transparent_white">
                 <color rgba="1 1 1 0.5" />
             </material>
@@ -134,5 +134,5 @@
         <collision>
             <geometry>
-               <mesh filename="led_1.obj" scale="1.5 1.5 1.5" />
+               <mesh filename="led_1.obj" scale=".5 .5 .5" />
             </geometry>
             <origin xyz="0 0 0" />
@@ -146,8 +146,8 @@
         <visual>
             <geometry>
-                <mesh filename="led_2.obj" scale="1.5 1.5 1.5" />
-            </geometry>
-            <origin xyz="0 0 0" />
-            <material name="white">
+                <mesh filename="led_2.obj" scale=".5 .5 .5" />
+            </geometry>
+            <origin xyz="0 0 0" />
+            <material name="transparent_white">
                 <color rgba="1 1 1 0.5" />
             </material>
@@ -155,5 +155,5 @@
         <collision>
             <geometry>
-               <mesh filename="led_2.obj" scale="1.5 1.5 1.5" />
+               <mesh filename="led_2.obj" scale=".5 .5 .5" />
             </geometry>
             <origin xyz="0 0 0" />
@@ -167,8 +167,8 @@
         <visual>
             <geometry>
-                <mesh filename="led_3.obj" scale="1.5 1.5 1.5" />
-            </geometry>
-            <origin xyz="0 0 0" />
-            <material name="white">
+                <mesh filename="led_3.obj" scale=".5 .5 .5" />
+            </geometry>
+            <origin xyz="0 0 0" />
+            <material name="transparent_white">
                 <color rgba="1 1 1 0.5" />
             </material>
@@ -176,5 +176,5 @@
         <collision>
             <geometry>
-               <mesh filename="led_3.obj" scale="1.5 1.5 1.5" />
+               <mesh filename="led_3.obj" scale=".5 .5 .5" />
             </geometry>
             <origin xyz="0 0 0" />
@@ -188,8 +188,8 @@
         <visual>
             <geometry>
-                <mesh filename="led_4.obj" scale="1.5 1.5 1.5" />
-            </geometry>
-            <origin xyz="0 0 0" />
-            <material name="white">
+                <mesh filename="led_4.obj" scale=".5 .5 .5" />
+            </geometry>
+            <origin xyz="0 0 0" />
+            <material name="transparent_white">
                 <color rgba="1 1 1 0.5" />
             </material>
@@ -197,5 +197,5 @@
         <collision>
             <geometry>
-               <mesh filename="led_4.obj" scale="1.5 1.5 1.5" />
+               <mesh filename="led_4.obj" scale=".5 .5 .5" />
             </geometry>
             <origin xyz="0 0 0" />
@@ -209,8 +209,8 @@
         <visual>
             <geometry>
-                <mesh filename="led_5.obj" scale="1.5 1.5 1.5" />
-            </geometry>
-            <origin xyz="0 0 0" />
-            <material name="white">
+                <mesh filename="led_5.obj" scale=".5 .5 .5" />
+            </geometry>
+            <origin xyz="0 0 0" />
+            <material name="transparent_white">
                 <color rgba="1 1 1 0.5" />
             </material>
@@ -218,5 +218,5 @@
         <collision>
             <geometry>
-               <mesh filename="led_5.obj" scale="1.5 1.5 1.5" />
+               <mesh filename="led_5.obj" scale=".5 .5 .5" />
             </geometry>
             <origin xyz="0 0 0" />
@@ -230,8 +230,8 @@
         <visual>
             <geometry>
-                <mesh filename="led_6.obj" scale="1.5 1.5 1.5" />
-            </geometry>
-            <origin xyz="0 0 0" />
-            <material name="white">
+                <mesh filename="led_6.obj" scale=".5 .5 .5" />
+            </geometry>
+            <origin xyz="0 0 0" />
+            <material name="transparent_white">
                 <color rgba="1 1 1 0.5" />
             </material>
@@ -239,5 +239,5 @@
         <collision>
             <geometry>
-               <mesh filename="led_6.obj" scale="1.5 1.5 1.5" />
+               <mesh filename="led_6.obj" scale=".5 .5 .5" />
             </geometry>
             <origin xyz="0 0 0" />
@@ -251,8 +251,8 @@
         <visual>
             <geometry>
-                <mesh filename="led_7.obj" scale="1.5 1.5 1.5" />
-            </geometry>
-            <origin xyz="0 0 0" />
-            <material name="white">
+                <mesh filename="led_7.obj" scale=".5 .5 .5" />
+            </geometry>
+            <origin xyz="0 0 0" />
+            <material name="transparent_white">
                 <color rgba="1 1 1 0.5" />
             </material>
@@ -260,5 +260,5 @@
         <collision>
             <geometry>
-               <mesh filename="led_7.obj" scale="1.5 1.5 1.5" />
+               <mesh filename="led_7.obj" scale=".5 .5 .5" />
             </geometry>
             <origin xyz="0 0 0" />
@@ -272,40 +272,40 @@
         <parent link="base_link" />
         <child link="led0" />
-        <origin rpy="1.57 0 -1.57" xyz="0.0 0 .1" />
+        <origin rpy="1.57 0 -1.5" xyz="-0.1 -0.01 0.12" />
     </joint>
     <joint name="base_to_led1" type="fixed">
         <parent link="base_link" />
         <child link="led1" />
-        <origin rpy="1.57 0 -1.5" xyz="0.0 0.0 .1" />
+        <origin rpy="1.57 0 -1.5" xyz="-0.1 -0.01 .12" />
     </joint>
     <joint name="base_to_led2" type="fixed">
         <parent link="base_link" />
         <child link="led2" />
-        <origin rpy="1.57 0 -1.43" xyz="0.0 0.0 .1" />
+        <origin rpy="1.57 0 -1.5" xyz="-0.1 -0.01 .12" />
     </joint>
     <joint name="base_to_led3" type="fixed">
         <parent link="base_link" />
         <child link="led3" />
-        <origin rpy="1.57 0 -1.37" xyz="0.0 0.0 .1" />
+        <origin rpy="1.57 0 -1.5" xyz="-0.1 -0.01 .12" />
     </joint>
     <joint name="base_to_led4" type="fixed">
         <parent link="base_link" />
         <child link="led4" />
-        <origin rpy="1.57 0 -1.31" xyz="0.0 0.0 .1" />
+        <origin rpy="1.57 0 -1.5" xyz="-0.1 -0.01 .12" />
     </joint>
     <joint name="base_to_led5" type="fixed">
         <parent link="base_link" />
         <child link="led5" />
-        <origin rpy="1.57 0 -1.25" xyz="0.0 0.0 .1" />
+        <origin rpy="1.57 0 -1.5" xyz="-0.1 -0.01 .12" />
     </joint>
     <joint name="base_to_led6" type="fixed">
         <parent link="base_link" />
         <child link="led6" />
-        <origin rpy="1.57 0 -1.19" xyz="0.0 0.0 .1" />
+        <origin rpy="1.57 0 -1.5" xyz="-0.1 -0.01 .12" />
     </joint>
     <joint name="base_to_led7" type="fixed">
         <parent link="base_link" />
         <child link="led7" />
-        <origin rpy="1.57 0 -1.13" xyz="0.0 0.0 .1" />
+        <origin rpy="1.57 0 -1.5" xyz="-0.1 -0.01 .12" />
     </joint>
     <link name="cam">
@@ -774,5 +774,5 @@
 			 <mesh filename="cone.obj" scale="1 1 1"/>
       </geometry>
-      <material name="red">
+      <material name="transparent_red">
         <color rgba="1 0 0 0."/>
       </material>
@@ -801,5 +801,5 @@
 			 <mesh filename="cone.obj" scale="1 1 1"/>
       </geometry>
-      <material name="red">
+      <material name="transparent_red">
         <color rgba="1 0 0 0"/>
       </material>
@@ -828,5 +828,5 @@
 			 <mesh filename="cone.obj" scale="1 1 1"/>
       </geometry>
-      <material name="red">
+      <material name="transparent_red">
         <color rgba="1 0 0 0"/>
       </material>
@@ -855,5 +855,5 @@
 			 <mesh filename="cone.obj" scale="1 1 1"/>
       </geometry>
-      <material name="red">
+      <material name="transparent_red">
         <color rgba="1 0 0 0"/>
       </material>
@@ -882,5 +882,5 @@
 			 <mesh filename="cone.obj" scale="1 1 1"/>
       </geometry>
-      <material name="red">
+      <material name="transparent_red">
         <color rgba="1 0 0 0"/>
       </material>
@@ -909,6 +909,6 @@
 			 <mesh filename="cone.obj" scale="1 1 1"/>
       </geometry>
-      <material name="red">
-        <color rgba="0 0 0 0"/>
+      <material name="transparent_red">
+        <color rgba="1 0 0 0"/>
       </material>
     </visual>
@@ -936,6 +936,6 @@
 			 <mesh filename="cone.obj" scale="1 1 1"/>
       </geometry>
-      <material name="red">
-        <color rgba="0 0 0 0"/>
+      <material name="transparent_red">
+        <color rgba="1 0 0 0"/>
       </material>
     </visual>
@@ -963,6 +963,6 @@
                 <mesh filename="cone.obj" scale="1 1 1"/>
         </geometry>
-        <material name="red">
-            <color rgba="0 0 0 0"/>
+        <material name="transparent_red">
+            <color rgba="1 0 0 0"/>
         </material>
         </visual>
@@ -990,6 +990,6 @@
 			 <mesh filename="cone.obj" scale="3 3 3"/>
       </geometry>
-      <material name="red">
-        <color rgba="0 0 0 0"/>
+      <material name="transparent_red">
+        <color rgba="1 0 0 0"/>
       </material>
     </visual>
@@ -1017,6 +1017,6 @@
 			 <mesh filename="cone.obj" scale="3 3 3"/>
       </geometry>
-      <material name="red">
-        <color rgba="0 0 0 0"/>
+      <material name="transparent_red">
+        <color rgba="1 0 0 0"/>
       </material>
     </visual>
@@ -1044,6 +1044,6 @@
 			 <mesh filename="cone.obj" scale="3 3 3"/>
       </geometry>
-      <material name="red">
-        <color rgba="0 0 0 0"/>
+      <material name="transparent_red">
+        <color rgba="1 0 0 0"/>
       </material>
     </visual>
@@ -1071,6 +1071,6 @@
 			 <mesh filename="cone.obj" scale="3 3 3"/>
       </geometry>
-      <material name="red">
-        <color rgba="0 0 0 0"/>
+      <material name="transparent_red">
+        <color rgba="1 0 0 0"/>
       </material>
     </visual>
@@ -1098,6 +1098,6 @@
 			 <mesh filename="cone.obj" scale="3 3 3"/>
       </geometry>
-      <material name="red">
-        <color rgba="0 0 0 0"/>
+      <material name="transparent_red">
+        <color rgba="1 0 0 0"/>
       </material>
     </visual>
@@ -1125,6 +1125,6 @@
 			 <mesh filename="cone.obj" scale="3 3 3"/>
       </geometry>
-      <material name="red">
-        <color rgba="0 0 0 0"/>
+      <material name="transparent_red">
+        <color rgba="1 0 0 0"/>
       </material>
     </visual>
@@ -1152,6 +1152,6 @@
 			 <mesh filename="cone.obj" scale="3 3 3"/>
       </geometry>
-      <material name="red">
-        <color rgba="0 0 0 0"/>
+      <material name="transparent_red">
+        <color rgba="1 0 0 0"/>
       </material>
     </visual>
@@ -1179,6 +1179,6 @@
             <mesh filename="cone.obj" scale="3 3 3"/>
         </geometry>
-        <material name="red">
-            <color rgba="0 0 0 0"/>
+        <material name="transparent_red">
+            <color rgba="1 0 0 0"/>
         </material>
         </visual>

Commit message: Light sensor step simplied (only 1 ray now). Ghost objects improved. Validated in braitenber example

File: spike_swarm_sim/models/entities/epuck/epuck.urdf.xacro (robot description, xacro)
@@ -21,5 +21,5 @@
         </inertial>
     </link>
-     <link name="right_wheel">
+    <link name="right_wheel">
         <visual>
             <geometry>
@@ -772,5 +772,5 @@
       <origin rpy="0 0 0" xyz="0 0 0"/>
       <geometry>
-			 <mesh filename="cone.obj" scale="1 1 1"/>
+			 <mesh filename="ghost_DS.obj" scale="1 1 1"/>
       </geometry>
       <material name="transparent_red">
@@ -780,5 +780,5 @@
      <collision>
             <geometry>
-            <mesh filename="cone.obj" scale="1 1 1"/>
+            <mesh filename="ghost_DS.obj" scale="1 1 1"/>
             </geometry>
             <origin xyz="0 0 0" />
@@ -799,5 +799,5 @@
       <origin rpy="0 0 0" xyz="0 0 0.0"/>
       <geometry>
-			 <mesh filename="cone.obj" scale="1 1 1"/>
+			 <mesh filename="ghost_DS.obj" scale="1 1 1"/>
       </geometry>
       <material name="transparent_red">
@@ -807,5 +807,5 @@
     <collision>
             <geometry>
-            <mesh filename="cone.obj" scale="1 1 1"/>
+            <mesh filename="ghost_DS.obj" scale="1 1 1"/>
             </geometry>
             <origin xyz="0 0 0" />
@@ -826,5 +826,5 @@
       <origin rpy="0 0 0" xyz="0 0 0.0"/>
       <geometry>
-			 <mesh filename="cone.obj" scale="1 1 1"/>
+			 <mesh filename="ghost_DS.obj" scale="1 1 1"/>
       </geometry>
       <material name="transparent_red">
@@ -834,5 +834,5 @@
          <collision>
             <geometry>
-            <mesh filename="cone.obj" scale="1 1 1"/>
+            <mesh filename="ghost_DS.obj" scale="1 1 1"/>
             </geometry>
             <origin xyz="0 0 0" />
@@ -853,5 +853,5 @@
       <origin rpy="0 0 0" xyz="0 0 0.0"/>
       <geometry>
-			 <mesh filename="cone.obj" scale="1 1 1"/>
+			 <mesh filename="ghost_DS.obj" scale="1 1 1"/>
       </geometry>
       <material name="transparent_red">
@@ -861,5 +861,5 @@
          <collision>
             <geometry>
-            <mesh filename="cone.obj" scale="1 1 1"/>
+            <mesh filename="ghost_DS.obj" scale="1 1 1"/>
             </geometry>
             <origin xyz="0 0 0" />
@@ -880,5 +880,5 @@
       <origin rpy="0 0 0" xyz="0 0 0"/>
       <geometry>
-			 <mesh filename="cone.obj" scale="1 1 1"/>
+			 <mesh filename="ghost_DS.obj" scale="1 1 1"/>
       </geometry>
       <material name="transparent_red">
@@ -888,5 +888,5 @@
          <collision>
             <geometry>
-            <mesh filename="cone.obj" scale="1 1 1"/>
+            <mesh filename="ghost_DS.obj" scale="1 1 1"/>
             </geometry>
             <origin xyz="0 0 0" />
@@ -907,5 +907,5 @@
       <origin rpy="0 0 0" xyz="0 0 0"/>
       <geometry>
-			 <mesh filename="cone.obj" scale="1 1 1"/>
+			 <mesh filename="ghost_DS.obj" scale="1 1 1"/>
       </geometry>
       <material name="transparent_red">
@@ -915,5 +915,5 @@
          <collision>
             <geometry>
-            <mesh filename="cone.obj" scale="1 1 1"/>
+            <mesh filename="ghost_DS.obj" scale="1 1 1"/>
             </geometry>
             <origin xyz="0 0 0" />
@@ -934,5 +934,5 @@
       <origin rpy="0 0 0" xyz="0 0 0"/>
       <geometry>
-			 <mesh filename="cone.obj" scale="1 1 1"/>
+			 <mesh filename="ghost_DS.obj" scale="1 1 1"/>
       </geometry>
       <material name="transparent_red">
@@ -942,5 +942,5 @@
          <collision>
             <geometry>
-            <mesh filename="cone.obj" scale="1 1 1"/>
+            <mesh filename="ghost_DS.obj" scale="1 1 1"/>
             </geometry>
             <origin xyz="0 0 0" />
@@ -961,5 +961,5 @@
         <origin rpy="0 0 0" xyz="0 0 0"/>
         <geometry>
-                <mesh filename="cone.obj" scale="1 1 1"/>
+                <mesh filename="ghost_DS.obj" scale="1 1 1"/>
         </geometry>
         <material name="transparent_red">
@@ -969,5 +969,5 @@
             <collision>
                 <geometry>
-                <mesh filename="cone.obj" scale="1 1 1"/>
+                <mesh filename="ghost_DS.obj" scale="1 1 1"/>
                 </geometry>
                 <origin xyz="0 0 0" />
@@ -988,5 +988,5 @@
       <origin rpy="0 0 0" xyz="0 0 0"/>
       <geometry>
-			 <mesh filename="cone.obj" scale="3 3 3"/>
+			 <mesh filename="ghost_LS.obj" scale="1 1 1"/>
       </geometry>
       <material name="transparent_red">
@@ -996,5 +996,5 @@
      <collision>
             <geometry>
-            <mesh filename="cone.obj" scale="3 3 3"/>
+            <mesh filename="ghost_LS.obj" scale="1 1 1"/>
             </geometry>
             <origin xyz="0 0 0" />
@@ -1015,5 +1015,5 @@
       <origin rpy="0 0 0" xyz="0 0 0.0"/>
       <geometry>
-			 <mesh filename="cone.obj" scale="3 3 3"/>
+			 <mesh filename="ghost_LS.obj" scale="1 1 1"/>
       </geometry>
       <material name="transparent_red">
@@ -1023,5 +1023,5 @@
     <collision>
             <geometry>
-            <mesh filename="cone.obj" scale="3 3 3"/>
+            <mesh filename="ghost_LS.obj" scale="1 1 1"/>
             </geometry>
             <origin xyz="0 0 0" />
@@ -1042,5 +1042,5 @@
       <origin rpy="0 0 0" xyz="0 0 0.0"/>
       <geometry>
-			 <mesh filename="cone.obj" scale="3 3 3"/>
+			 <mesh filename="ghost_LS.obj" scale="1 1 1"/>
       </geometry>
       <material name="transparent_red">
@@ -1050,5 +1050,5 @@
          <collision>
             <geometry>
-            <mesh filename="cone.obj" scale="3 3 3"/>
+            <mesh filename="ghost_LS.obj" scale="1 1 1"/>
             </geometry>
             <origin xyz="0 0 0" />
@@ -1069,5 +1069,5 @@
       <origin rpy="0 0 0" xyz="0 0 0.0"/>
       <geometry>
-			 <mesh filename="cone.obj" scale="3 3 3"/>
+			 <mesh filename="ghost_LS.obj" scale="1 1 1"/>
       </geometry>
       <material name="transparent_red">
@@ -1096,5 +1096,5 @@
       <origin rpy="0 0 0" xyz="0 0 0"/>
       <geometry>
-			 <mesh filename="cone.obj" scale="3 3 3"/>
+			 <mesh filename="ghost_LS.obj" scale="1 1 1"/>
       </geometry>
       <material name="transparent_red">
@@ -1104,5 +1104,5 @@
          <collision>
             <geometry>
-            <mesh filename="cone.obj" scale="3 3 3"/>
+            <mesh filename="ghost_LS.obj" scale="1 1 1"/>
             </geometry>
             <origin xyz="0 0 0" />
@@ -1123,5 +1123,5 @@
       <origin rpy="0 0 0" xyz="0 0 0"/>
       <geometry>
-			 <mesh filename="cone.obj" scale="3 3 3"/>
+			 <mesh filename="ghost_LS.obj" scale="1 1 1"/>
       </geometry>
       <material name="transparent_red">
@@ -1131,5 +1131,5 @@
          <collision>
             <geometry>
-            <mesh filename="cone.obj" scale="3 3 3"/>
+            <mesh filename="ghost_LS.obj" scale="1 1 1"/>
             </geometry>
             <origin xyz="0 0 0" />
@@ -1150,13 +1150,13 @@
       <origin rpy="0 0 0" xyz="0 0 0"/>
       <geometry>
-			 <mesh filename="cone.obj" scale="3 3 3"/>
-      </geometry>
-      <material name="transparent_red">
-        <color rgba="1 0 0 0"/>
-      </material>
-    </visual>
-        <collision>
-            <geometry>
-                <mesh filename="cone.obj" scale="3 3 3"/>
+			 <mesh filename="ghost_LS.obj" scale="1 1 1"/>
+      </geometry>
+      <material name="transparent_red">
+        <color rgba="1 0 0 0"/>
+      </material>
+    </visual>
+        <collision>
+            <geometry>
+                <mesh filename="ghost_LS.obj" scale="1 1 1"/>
             </geometry>
             <origin xyz="0 0 0" />
@@ -1177,5 +1177,5 @@
         <origin rpy="0 0 0" xyz="0 0 0"/>
         <geometry>
-            <mesh filename="cone.obj" scale="3 3 3"/>
+            <mesh filename="ghost_LS.obj" scale="1 1 1"/>
         </geometry>
         <material name="transparent_red">
@@ -1185,5 +1185,5 @@
             <collision>
                 <geometry>
-                <mesh filename="cone.obj" scale="3 3 3"/>
+                <mesh filename="ghost_LS.obj" scale="1 1 1"/>
                 </geometry>
                 <origin xyz="0 0 0" />

File: spike_swarm_sim/models/entities/light_source/light.urdf (robot description, URDF)
Before this commit: robot light, 1 links, 0 joints
Links:
- link baseLink: geometry collision mesh filename=sphere.obj scale=0.3 0.3 0.3; visual mesh filename=sphere.obj scale=0.3 0.3 0.3
