Commit message: Simulation speeded up. Sensors (DS and LS) improved.

File: mereli/models/entities/epuck/epuck.urdf (robot description, URDF)
Before this commit: robot epuck, 23 links, 22 joints
Links:
- added link ghost_cone_LS0, mass 0.0; collision mesh filename=ghost_LS.obj scale=1 1 1; visual mesh filename=ghost_LS.obj scale=1 1 1
- added link ghost_cone_LS1, mass 0.0; collision mesh filename=ghost_LS.obj scale=1 1 1; visual mesh filename=ghost_LS.obj scale=1 1 1
- added link ghost_cone_LS2, mass 0.0; collision mesh filename=ghost_LS.obj scale=1 1 1; visual mesh filename=ghost_LS.obj scale=1 1 1
- added link ghost_cone_LS3, mass 0.0; collision mesh filename=cone.obj scale=3 3 3; visual mesh filename=ghost_LS.obj scale=1 1 1
- added link ghost_cone_LS4, mass 0.0; collision mesh filename=ghost_LS.obj scale=1 1 1; visual mesh filename=ghost_LS.obj scale=1 1 1
- added link ghost_cone_LS5, mass 0.0; collision mesh filename=ghost_LS.obj scale=1 1 1; visual mesh filename=ghost_LS.obj scale=1 1 1
- added link ghost_cone_LS6, mass 0.0; collision mesh filename=ghost_LS.obj scale=1 1 1; visual mesh filename=ghost_LS.obj scale=1 1 1
- added link ghost_cone_LS7, mass 0.0; collision mesh filename=ghost_LS.obj scale=1 1 1; visual mesh filename=ghost_LS.obj scale=1 1 1
- added link led1, mass 0.01; collision mesh filename=led_1.obj scale=.5 .5 .5; visual mesh filename=led_1.obj scale=.5 .5 .5
- added link led2, mass 0.01; collision mesh filename=led_2.obj scale=.5 .5 .5; visual mesh filename=led_2.obj scale=.5 .5 .5
- added link led3, mass 0.01; collision mesh filename=led_3.obj scale=.5 .5 .5; visual mesh filename=led_3.obj scale=.5 .5 .5
- added link led4, mass 0.01; collision mesh filename=led_4.obj scale=.5 .5 .5; visual mesh filename=led_4.obj scale=.5 .5 .5
- added link led5, mass 0.01; collision mesh filename=led_5.obj scale=.5 .5 .5; visual mesh filename=led_5.obj scale=.5 .5 .5
- added link led6, mass 0.01; collision mesh filename=led_6.obj scale=.5 .5 .5; visual mesh filename=led_6.obj scale=.5 .5 .5
- added link led7, mass 0.01; collision mesh filename=led_7.obj scale=.5 .5 .5; visual mesh filename=led_7.obj scale=.5 .5 .5
- link arrow: geometry visual mesh filename=arrow.obj scale=0.1 0.1 0.1
- link ghost_cone_DS0: geometry collision mesh filename=ghost_DS.obj scale=0.5 0.5 0.5; visual mesh filename=ghost_DS.obj scale=0.5 0.5 0.5
- link ghost_cone_DS1: geometry collision mesh filename=ghost_DS.obj scale=0.5 0.5 0.5; visual mesh filename=ghost_DS.obj scale=0.5 0.5 0.5
- link ghost_cone_DS2: geometry collision mesh filename=ghost_DS.obj scale=0.5 0.5 0.5; visual mesh filename=ghost_DS.obj scale=0.5 0.5 0.5
- link ghost_cone_DS3: geometry collision mesh filename=ghost_DS.obj scale=0.5 0.5 0.5; visual mesh filename=ghost_DS.obj scale=0.5 0.5 0.5
- link ghost_cone_DS4: geometry collision mesh filename=ghost_DS.obj scale=.5 .5 .5; visual mesh filename=ghost_DS.obj scale=.5 .5 .5
- link ghost_cone_DS5: geometry collision mesh filename=ghost_DS.obj scale=.5 .5 .5; visual mesh filename=ghost_DS.obj scale=.5 .5 .5
- link ghost_cone_DS6: geometry collision mesh filename=ghost_DS.obj scale=.5 .5 .5; visual mesh filename=ghost_DS.obj scale=.5 .5 .5
- link ghost_cone_DS7: geometry collision mesh filename=ghost_DS.obj scale=.5 .5 .5; visual mesh filename=ghost_DS.obj scale=.5 .5 ..5
- link led0: geometry collision mesh filename=led_0.obj scale=.5 .5 .5; visual mesh filename=led_0.obj scale=.5 .5 .5
Joints:
- added joint IR0_to_ghost_cone_LS0: type fixed, parent IR0, child ghost_cone_LS0, origin xyz=0 0.0 0.0 rpy=-1.57 0.4 1.57
- added joint IR1_to_ghost_cone_LS1: type fixed, parent IR1, child ghost_cone_LS1, origin xyz=0 0.0 0.0 rpy=-1.57 0.4 1.57
- added joint IR2_to_ghost_cone_LS2: type fixed, parent IR2, child ghost_cone_LS2, origin xyz=0 0.0 0.0 rpy=-1.57 0.4 1.57
- added joint IR3_to_ghost_cone_LS3: type fixed, parent IR3, child ghost_cone_LS3, origin xyz=0 0.0 0.0 rpy=-1.57 0.4 1.57
- added joint IR4_to_ghost_cone_LS4: type fixed, parent IR4, child ghost_cone_LS4, origin xyz=0 0.0 0.0 rpy=-1.57 0.4 1.57
- added joint IR5_to_ghost_cone_LS5: type fixed, parent IR5, child ghost_cone_LS5, origin xyz=0 0.0 0.0 rpy=-1.57 0.4 1.57
- added joint IR6_to_ghost_cone_LS6: type fixed, parent IR6, child ghost_cone_LS6, origin xyz=0 0.0 0.0 rpy=-1.57 0.4 1.57
- added joint IR7_to_ghost_cone_LS7: type fixed, parent IR7, child ghost_cone_LS7, origin xyz=0 0.0 0.0 rpy=-1.57 0.4 1.57
- added joint base_to_led1: type fixed, parent base_link, child led1, origin xyz=-0.1 -0.01 .12 rpy=1.57 0 -1.5
- added joint base_to_led2: type fixed, parent base_link, child led2, origin xyz=-0.1 -0.01 .12 rpy=1.57 0 -1.5
- added joint base_to_led3: type fixed, parent base_link, child led3, origin xyz=-0.1 -0.01 .12 rpy=1.57 0 -1.5
- added joint base_to_led4: type fixed, parent base_link, child led4, origin xyz=-0.1 -0.01 .12 rpy=1.57 0 -1.5
- added joint base_to_led5: type fixed, parent base_link, child led5, origin xyz=-0.1 -0.01 .12 rpy=1.57 0 -1.5
- added joint base_to_led6: type fixed, parent base_link, child led6, origin xyz=-0.1 -0.01 .12 rpy=1.57 0 -1.5
- added joint base_to_led7: type fixed, parent base_link, child led7, origin xyz=-0.1 -0.01 .12 rpy=1.57 0 -1.5
- joint base_to_led0: origin xyz=0 -0.098 0.12 rpy=1.57075 0 0 -> xyz=-0.1 -0.01 0.12 rpy=1.57 0 -1.5

File: mereli/models/entities/epuck/epuck.urdf.xacro (robot description, xacro)
@@ -326,5 +326,5 @@
         </collision>
         <inertial>
-            <mass value="0.005" />
+            <mass value="0.00" />
             <inertia ixx="1.0" ixy="0.0" ixz="0.0" iyy="1.0" iyz="0.0" izz="1.0" />
         </inertial>
@@ -747,10 +747,4 @@
             </material>
         </visual>
-        <collision>
-            <geometry>
-               <mesh filename="arrow.obj" scale="0.1 0.1 0.1"/>
-            </geometry>
-            <origin xyz="0 0 0" rpy="1.57 0 -1.57"/>
-        </collision>
         <inertial>
             <mass value="0"/>
