Commit message: Sensor step slightly speed up

File: mereli/models/entities/epuck/epuck.urdf.xacro (robot description, xacro)
@@ -772,5 +772,5 @@
       <origin rpy="0 0 0" xyz="0 0 0"/>
       <geometry>
-			 <mesh filename="ghost_DS.obj" scale="1 1 1"/>
+			 <mesh filename="ghost_DS.obj" scale="0.5 0.5 0.5"/>
       </geometry>
       <material name="transparent_red">
@@ -780,5 +780,5 @@
      <collision>
             <geometry>
-            <mesh filename="ghost_DS.obj" scale="1 1 1"/>
+            <mesh filename="ghost_DS.obj" scale="0.5 0.5 0.5"/>
             </geometry>
             <origin xyz="0 0 0" />
@@ -799,5 +799,5 @@
       <origin rpy="0 0 0" xyz="0 0 0.0"/>
       <geometry>
-			 <mesh filename="ghost_DS.obj" scale="1 1 1"/>
+			 <mesh filename="ghost_DS.obj" scale="0.5 0.5 0.5"/>
       </geometry>
       <material name="transparent_red">
@@ -807,5 +807,5 @@
     <collision>
             <geometry>
-            <mesh filename="ghost_DS.obj" scale="1 1 1"/>
+            <mesh filename="ghost_DS.obj" scale="0.5 0.5 0.5"/>
             </geometry>
             <origin xyz="0 0 0" />
@@ -826,5 +826,5 @@
       <origin rpy="0 0 0" xyz="0 0 0.0"/>
       <geometry>
-			 <mesh filename="ghost_DS.obj" scale="1 1 1"/>
+			 <mesh filename="ghost_DS.obj" scale="0.5 0.5 0.5"/>
       </geometry>
       <material name="transparent_red">
@@ -834,5 +834,5 @@
          <collision>
             <geometry>
-            <mesh filename="ghost_DS.obj" scale="1 1 1"/>
+            <mesh filename="ghost_DS.obj" scale="0.5 0.5 0.5"/>
             </geometry>
             <origin xyz="0 0 0" />
@@ -853,5 +853,5 @@
       <origin rpy="0 0 0" xyz="0 0 0.0"/>
       <geometry>
-			 <mesh filename="ghost_DS.obj" scale="1 1 1"/>
+			 <mesh filename="ghost_DS.obj" scale="0.5 0.5 0.5"/>
       </geometry>
       <material name="transparent_red">
@@ -861,5 +861,5 @@
          <collision>
             <geometry>
-            <mesh filename="ghost_DS.obj" scale="1 1 1"/>
+            <mesh filename="ghost_DS.obj" scale="0.5 0.5 0.5"/>
             </geometry>
             <origin xyz="0 0 0" />
@@ -880,5 +880,5 @@
       <origin rpy="0 0 0" xyz="0 0 0"/>
       <geometry>
-			 <mesh filename="ghost_DS.obj" scale="1 1 1"/>
+			 <mesh filename="ghost_DS.obj" scale=".5 .5 .5"/>
       </geometry>
       <material name="transparent_red">
@@ -888,5 +888,5 @@
          <collision>
             <geometry>
-            <mesh filename="ghost_DS.obj" scale="1 1 1"/>
+            <mesh filename="ghost_DS.obj" scale=".5 .5 .5"/>
             </geometry>
             <origin xyz="0 0 0" />
@@ -907,5 +907,5 @@
       <origin rpy="0 0 0" xyz="0 0 0"/>
       <geometry>
-			 <mesh filename="ghost_DS.obj" scale="1 1 1"/>
+			 <mesh filename="ghost_DS.obj" scale=".5 .5 .5"/>
       </geometry>
       <material name="transparent_red">
@@ -915,5 +915,5 @@
          <collision>
             <geometry>
-            <mesh filename="ghost_DS.obj" scale="1 1 1"/>
+            <mesh filename="ghost_DS.obj" scale=".5 .5 .5"/>
             </geometry>
             <origin xyz="0 0 0" />
@@ -934,5 +934,5 @@
       <origin rpy="0 0 0" xyz="0 0 0"/>
       <geometry>
-			 <mesh filename="ghost_DS.obj" scale="1 1 1"/>
+			 <mesh filename="ghost_DS.obj" scale=".5 .5 .5"/>
       </geometry>
       <material name="transparent_red">
@@ -942,5 +942,5 @@
          <collision>
             <geometry>
-            <mesh filename="ghost_DS.obj" scale="1 1 1"/>
+            <mesh filename="ghost_DS.obj" scale=".5 .5 .5"/>
             </geometry>
             <origin xyz="0 0 0" />
@@ -961,5 +961,5 @@
         <origin rpy="0 0 0" xyz="0 0 0"/>
         <geometry>
-                <mesh filename="ghost_DS.obj" scale="1 1 1"/>
+                <mesh filename="ghost_DS.obj" scale=".5 .5 ..5"/>
         </geometry>
         <material name="transparent_red">
@@ -969,5 +969,5 @@
             <collision>
                 <geometry>
-                <mesh filename="ghost_DS.obj" scale="1 1 1"/>
+                <mesh filename="ghost_DS.obj" scale=".5 .5 .5"/>
                 </geometry>
                 <origin xyz="0 0 0" />

Commit message: Epuck realistic dimensions and mass fixed. Few config changes.

File: mereli/models/entities/epuck/epuck.urdf.xacro (robot description, xacro)
@@ -17,5 +17,5 @@
         </collision>
         <inertial>
-            <mass value="1.5" />
+            <mass value="0.1" />
             <inertia ixx="1.0" ixy="0.0" ixz="0.0" iyy="1.0" iyz="0.0" izz="1.0" />
         </inertial>
@@ -38,5 +38,5 @@
         </collision>
         <inertial>
-            <mass value="0.1" />
+            <mass value="0.025" />
             <inertia ixx="1.0" ixy="0.0" ixz="0.0" iyy="1.0" iyz="0.0" izz="1.0" />
         </inertial>
@@ -59,5 +59,5 @@
         </collision>
         <inertial>
-            <mass value="0.1" />
+            <mass value="0.025" />
             <inertia ixx="1.0" ixy="0.0" ixz="0.0" iyy="1.0" iyz="0.0" izz="1.0" />
         </inertial>
@@ -92,5 +92,5 @@
         </collision>
         <inertial>
-            <mass value="0.5" />
+            <mass value="0.025" />
             <inertia ixx="1.0" ixy="0.0" ixz="0.0" iyy="1.0" iyz="0.0" izz="1.0" />
         </inertial>
@@ -118,5 +118,5 @@
         </collision>
         <inertial>
-            <mass value="0.01" />
+            <mass value="0.0" />
             <inertia ixx="1.0" ixy="0.0" ixz="0.0" iyy="1.0" iyz="0.0" izz="1.0" />
         </inertial>
@@ -139,5 +139,5 @@
         </collision>
         <inertial>
-            <mass value="0.01" />
+            <mass value="0.0" />
             <inertia ixx="1.0" ixy="0.0" ixz="0.0" iyy="1.0" iyz="0.0" izz="1.0" />
         </inertial>
@@ -160,5 +160,5 @@
         </collision>
         <inertial>
-            <mass value="0.01" />
+            <mass value="0.0" />
             <inertia ixx="1.0" ixy="0.0" ixz="0.0" iyy="1.0" iyz="0.0" izz="1.0" />
         </inertial>
@@ -181,5 +181,5 @@
         </collision>
         <inertial>
-            <mass value="0.01" />
+            <mass value="0.00" />
             <inertia ixx="1.0" ixy="0.0" ixz="0.0" iyy="1.0" iyz="0.0" izz="1.0" />
         </inertial>
@@ -202,5 +202,5 @@
         </collision>
         <inertial>
-            <mass value="0.01" />
+            <mass value="0.0" />
             <inertia ixx="1.0" ixy="0.0" ixz="0.0" iyy="1.0" iyz="0.0" izz="1.0" />
         </inertial>
@@ -223,5 +223,5 @@
         </collision>
         <inertial>
-            <mass value="0.01" />
+            <mass value="0.0" />
             <inertia ixx="1.0" ixy="0.0" ixz="0.0" iyy="1.0" iyz="0.0" izz="1.0" />
         </inertial>
@@ -244,5 +244,5 @@
         </collision>
         <inertial>
-            <mass value="0.01" />
+            <mass value="0.0" />
             <inertia ixx="1.0" ixy="0.0" ixz="0.0" iyy="1.0" iyz="0.0" izz="1.0" />
         </inertial>
@@ -265,5 +265,5 @@
         </collision>
         <inertial>
-            <mass value="0.01" />
+            <mass value="0.0" />
             <inertia ixx="1.0" ixy="0.0" ixz="0.0" iyy="1.0" iyz="0.0" izz="1.0" />
         </inertial>

Commit message: Fixed serious bug with the DS ghost objs. New exp IR_COmm_1 ready to use.

File: mereli/models/entities/epuck/epuck.urdf.xacro (robot description, xacro)
@@ -769,5 +769,5 @@
       </geometry>
       <material name="transparent_red">
-        <color rgba="1 0 0 0."/>
+        <color rgba="1 0 0 0.0"/>
       </material>
     </visual>
@@ -782,5 +782,5 @@
         <parent link="IR0"/>
         <child link="ghost_cone_DS0"/>
-        <origin xyz="0 0.0 0.0" rpy="-1.57 0.3 1.57"/>
+        <origin xyz="0 0.0 0.0" rpy="-1.57 0.3 0"/>
     </joint>
     <link name="ghost_cone_DS1">
@@ -809,5 +809,5 @@
         <parent link="IR1"/>
         <child link="ghost_cone_DS1"/>
-        <origin xyz="0 0.0 0.0" rpy="-1.57 0.3 1.57"/>
+        <origin xyz="0 0.0 0.0" rpy="-1.57 0.3 0"/>
     </joint>
     <link name="ghost_cone_DS2">
@@ -836,5 +836,5 @@
         <parent link="IR2"/>
         <child link="ghost_cone_DS2"/>
-        <origin xyz="0 0.0 0.0" rpy="-1.57 0.3 1.57"/>
+        <origin xyz="0 0.0 0.0" rpy="-1.57 0.3 0"/>
     </joint>
     <link name="ghost_cone_DS3">
@@ -863,5 +863,5 @@
         <parent link="IR3"/>
         <child link="ghost_cone_DS3"/>
-        <origin xyz="0 0.0 0.0" rpy="-1.57 0.3 1.57"/>
+        <origin xyz="0 0.0 0.0" rpy="-1.57 0.3 0"/>
     </joint>
     <link name="ghost_cone_DS4">
@@ -890,5 +890,5 @@
         <parent link="IR4"/>
         <child link="ghost_cone_DS4"/>
-        <origin xyz="0 0.0 0.0" rpy="-1.57 0.3 1.57"/>
+        <origin xyz="0 0.0 0.0" rpy="-1.57 0.3 0"/>
     </joint>
     <link name="ghost_cone_DS5">
@@ -917,5 +917,5 @@
         <parent link="IR5"/>
         <child link="ghost_cone_DS5"/>
-        <origin xyz="0 0.0 0.0" rpy="-1.57 0.3 1.57"/>
+        <origin xyz="0 0.0 0.0" rpy="-1.57 0.3 0"/>
     </joint>
 <link name="ghost_cone_DS6">
@@ -944,5 +944,5 @@
         <parent link="IR6"/>
         <child link="ghost_cone_DS6"/>
-        <origin xyz="0 0.0 0.0" rpy="-1.57 0.3 1.57"/>
+        <origin xyz="0 0.0 0.0" rpy="-1.57 0.3 0"/>
     </joint>
     <link name="ghost_cone_DS7">
@@ -971,5 +971,5 @@
         <parent link="IR7"/>
         <child link="ghost_cone_DS7"/>
-        <origin xyz="0 0.0 0.0" rpy="-1.57 0.3 1.57"/>
+        <origin xyz="0 0.0 0.0" rpy="-1.57 0.3 0"/>
     </joint>
     <link name="ghost_cone_LS0">

Commit message: Multiple major changes: optimization of times, sensor readings, etc

File: mereli/models/entities/epuck/epuck.urdf.xacro (robot description, xacro)
@@ -583,46 +583,4 @@
             <origin xyz="0 0 0" rpy="0 0 6.0213"/>
             <ghost link='ghost_cone_DS7'/>
-        </sector>
-    </sensor>
-    <sensor name="light_sensor">
-       <sector index="0">
-            <parent link="IR0"/>
-            <origin xyz="0 0 0" rpy="0 0 0.26179"/>
-            <ghost link='ghost_cone_LS0'/>
-        </sector>
-        <sector index="1">
-            <parent link="IR1"/>
-            <origin xyz="0 0 0" rpy="0 0 0.78539"/>
-            <ghost link='ghost_cone_LS1'/>
-        </sector>
-        <sector index="2">
-            <parent link="IR2"/>
-            <origin xyz="0 0 0" rpy="0 0 1.57079"/>
-            <ghost link='ghost_cone_LS2'/>
-        </sector>
-        <sector index="3">
-            <parent link="IR3"/>
-            <origin xyz="0 0 0" rpy="0 0 2.61799"/>
-            <ghost link='ghost_cone_LS3'/>
-        </sector>
-        <sector index="4">
-            <parent link="IR4"/>
-            <origin xyz="0 0 0" rpy="0 0 3.66519"/>
-            <ghost link='ghost_cone_LS4'/>
-        </sector>
-        <sector index="5">
-            <parent link="IR5"/>
-            <origin xyz="0 0 0" rpy="0 0 4.71238"/>
-            <ghost link='ghost_cone_LS5'/>
-        </sector>
-        <sector index="6">
-            <parent link="IR6"/>
-            <origin xyz="0 0 0" rpy="0 0 5.49778"/>
-            <ghost link='ghost_cone_LS6'/>
-        </sector>
-        <sector index="7">
-            <parent link="IR7"/>
-            <origin xyz="0 0 0" rpy="0 0 6.0213"/>
-            <ghost link='ghost_cone_LS7'/>
         </sector>
     </sensor>
@@ -973,219 +931,3 @@
         <origin xyz="0 0.0 0.0" rpy="-1.57 0.3 0"/>
     </joint>
-    <link name="ghost_cone_LS0">
-    <inertial>
-      <origin rpy="0 0 0" xyz="0 0 0"/>
-       <mass value="0.0"/>
-       <inertia ixx="0" ixy="0" ixz="0" iyy="0" iyz="0" izz="0"/>
-    </inertial>
-    <visual>
-      <origin rpy="0 0 0" xyz="0 0 0"/>
-      <geometry>
-			 <mesh filename="ghost_LS.obj" scale="1 1 1"/>
-      </geometry>
-      <material name="transparent_red">
-        <color rgba="1 0 0 0"/>
-      </material>
-    </visual>
-     <collision>
-            <geometry>
-            <mesh filename="ghost_LS.obj" scale="1 1 1"/>
-            </geometry>
-            <origin xyz="0 0 0" />
-    </collision>
-    </link>
-    <joint name="IR0_to_ghost_cone_LS0" type="fixed">
-        <parent link="IR0"/>
-        <child link="ghost_cone_LS0"/>
-        <origin xyz="0 0.0 0.0" rpy="-1.57 0.4 1.57"/>
-    </joint>
-    <link name="ghost_cone_LS1">
-    <inertial>
-      <origin rpy="0 0 0" xyz="0 0 0"/>
-       <mass value="0.0"/>
-       <inertia ixx="0" ixy="0" ixz="0" iyy="0" iyz="0" izz="0"/>
-    </inertial>
-    <visual>
-      <origin rpy="0 0 0" xyz="0 0 0.0"/>
-      <geometry>
-			 <mesh filename="ghost_LS.obj" scale="1 1 1"/>
-      </geometry>
-      <material name="transparent_red">
-        <color rgba="1 0 0 0"/>
-      </material>
-    </visual>
-    <collision>
-            <geometry>
-            <mesh filename="ghost_LS.obj" scale="1 1 1"/>
-            </geometry>
-            <origin xyz="0 0 0" />
-    </collision>
-  </link>
-    <joint name="IR1_to_ghost_cone_LS1" type="fixed">
-        <parent link="IR1"/>
-        <child link="ghost_cone_LS1"/>
-        <origin xyz="0 0.0 0.0" rpy="-1.57 0.4 1.57"/>
-    </joint>
-    <link name="ghost_cone_LS2">
-    <inertial>
-      <origin rpy="0 0 0" xyz="0 0 0"/>
-       <mass value="0.0"/>
-       <inertia ixx="0" ixy="0" ixz="0" iyy="0" iyz="0" izz="0"/>
-    </inertial>
-    <visual>
-      <origin rpy="0 0 0" xyz="0 0 0.0"/>
-      <geometry>
-			 <mesh filename="ghost_LS.obj" scale="1 1 1"/>
-      </geometry>
-      <material name="transparent_red">
-        <color rgba="1 0 0 0"/>
-      </material>
-    </visual>
-         <collision>
-            <geometry>
-            <mesh filename="ghost_LS.obj" scale="1 1 1"/>
-            </geometry>
-            <origin xyz="0 0 0" />
-    </collision>
-    </link>
-    <joint name="IR2_to_ghost_cone_LS2" type="fixed">
-        <parent link="IR2"/>
-        <child link="ghost_cone_LS2"/>
-        <origin xyz="0 0.0 0.0" rpy="-1.57 0.4 1.57"/>
-    </joint>
-    <link name="ghost_cone_LS3">
-    <inertial>
-      <origin rpy="0 0 0" xyz="0 0 0"/>
-       <mass value="0.0"/>
-       <inertia ixx="0" ixy="0" ixz="0" iyy="0" iyz="0" izz="0"/>
-    </inertial>
-    <visual>
-      <origin rpy="0 0 0" xyz="0 0 0.0"/>
-      <geometry>
-			 <mesh filename="ghost_LS.obj" scale="1 1 1"/>
-      </geometry>
-      <material name="transparent_red">
-        <color rgba="1 0 0 0"/>
-      </material>
-    </visual>
-         <collision>
-            <geometry>
-            <mesh filename="cone.obj" scale="3 3 3"/>
-            </geometry>
-            <origin xyz="0 0 0" />
-    </collision>
-  </link>
-    <joint name="IR3_to_ghost_cone_LS3" type="fixed">
-        <parent link="IR3"/>
-        <child link="ghost_cone_LS3"/>
-        <origin xyz="0 0.0 0.0" rpy="-1.57 0.4 1.57"/>
-    </joint>
-    <link name="ghost_cone_LS4">
-    <inertial>
-      <origin rpy="0 0 0" xyz="0 0 0"/>
-       <mass value="0.0"/>
-       <inertia ixx="0" ixy="0" ixz="0" iyy="0" iyz="0" izz="0"/>
-    </inertial>
-    <visual>
-      <origin rpy="0 0 0" xyz="0 0 0"/>
-      <geometry>
-			 <mesh filename="ghost_LS.obj" scale="1 1 1"/>
-      </geometry>
-      <material name="transparent_red">
-        <color rgba="1 0 0 0"/>
-      </material>
-    </visual>
-         <collision>
-            <geometry>
-            <mesh filename="ghost_LS.obj" scale="1 1 1"/>
-            </geometry>
-            <origin xyz="0 0 0" />
-    </collision>
-    </link>
-    <joint name="IR4_to_ghost_cone_LS4" type="fixed">
-        <parent link="IR4"/>
-        <child link="ghost_cone_LS4"/>
-        <origin xyz="0 0.0 0.0" rpy="-1.57 0.4 1.57"/>
-    </joint>
-    <link name="ghost_cone_LS5">
-    <inertial>
-      <origin rpy="0 0 0" xyz="0 0 0"/>
-       <mass value="0.0"/>
-       <inertia ixx="0" ixy="0" ixz="0" iyy="0" iyz="0" izz="0"/>
-    </inertial>
-    <visual>
-      <origin rpy="0 0 0" xyz="0 0 0"/>
-      <geometry>
-			 <mesh filename="ghost_LS.obj" scale="1 1 1"/>
-      </geometry>
-      <material name="transparent_red">
-        <color rgba="1 0 0 0"/>
-      </material>
-    </visual>
-         <collision>
-            <geometry>
-            <mesh filename="ghost_LS.obj" scale="1 1 1"/>
-            </geometry>
-            <origin xyz="0 0 0" />
-    </collision>
-    </link>
-    <joint name="IR5_to_ghost_cone_LS5" type="fixed">
-        <parent link="IR5"/>
-        <child link="ghost_cone_LS5"/>
-        <origin xyz="0 0.0 0.0" rpy="-1.57 0.4 1.57"/>
-    </joint>
-<link name="ghost_cone_LS6">
-    <inertial>
-      <origin rpy="0 0 0" xyz="0 0 0"/>
-       <mass value="0.0"/>
-       <inertia ixx="0" ixy="0" ixz="0" iyy="0" iyz="0" izz="0"/>
-    </inertial>
-    <visual>
-      <origin rpy="0 0 0" xyz="0 0 0"/>
-      <geometry>
-			 <mesh filename="ghost_LS.obj" scale="1 1 1"/>
-      </geometry>
-      <material name="transparent_red">
-        <color rgba="1 0 0 0"/>
-      </material>
-    </visual>
-        <collision>
-            <geometry>
-                <mesh filename="ghost_LS.obj" scale="1 1 1"/>
-            </geometry>
-            <origin xyz="0 0 0" />
-        </collision>
-    </link>
-    <joint name="IR6_to_ghost_cone_LS6" type="fixed">
-        <parent link="IR6"/>
-        <child link="ghost_cone_LS6"/>
-        <origin xyz="0 0.0 0.0" rpy="-1.57 0.4 1.57"/>
-    </joint>
-    <link name="ghost_cone_LS7">
-        <inertial>
-        <origin rpy="0 0 0" xyz="0 0 0"/>
-        <mass value="0.0"/>
-        <inertia ixx="0" ixy="0" ixz="0" iyy="0" iyz="0" izz="0"/>
-        </inertial>
-        <visual>
-        <origin rpy="0 0 0" xyz="0 0 0"/>
-        <geometry>
-            <mesh filename="ghost_LS.obj" scale="1 1 1"/>
-        </geometry>
-        <material name="transparent_red">
-            <color rgba="1 0 0 0"/>
-        </material>
-        </visual>
-            <collision>
-                <geometry>
-                <mesh filename="ghost_LS.obj" scale="1 1 1"/>
-                </geometry>
-                <origin xyz="0 0 0" />
-        </collision>
-    </link>
-    <joint name="IR7_to_ghost_cone_LS7" type="fixed">
-        <parent link="IR7"/>
-        <child link="ghost_cone_LS7"/>
-        <origin xyz="0 0.0 0.0" rpy="-1.57 0.4 1.57"/>
-    </joint>
 </robot>
