Commit message: New formation comm space. New animations. IRIN experiments updated

File: mereli/models/entities/epuck/epuck_simple.urdf (robot description, URDF)
Before this commit: robot epuck, 30 links, 29 joints
Links:
- removed link arrow
- removed link cam
- removed link led0
- removed link led1
- removed link led2
- removed link led3
- removed link led4
- removed link led5
- removed link led6
- removed link led7
- removed link top
- link IR0: geometry collision box size=0.01 0.01 0.01; visual box size=0.01 0.01 0.01
- link IR1: geometry collision box size=0.01 0.01 0.01; visual box size=0.01 0.01 0.01
- link IR2: geometry collision box size=0.01 0.01 0.01; visual box size=0.01 0.01 0.01
- link IR3: geometry collision box size=0.01 0.01 0.01; visual box size=0.01 0.01 0.01
- link IR4: geometry collision box size=0.01 0.01 0.01; visual box size=0.01 0.01 0.01
- link IR5: geometry collision box size=0.01 0.01 0.01; visual box size=0.01 0.01 0.01
- link IR6: geometry collision box size=0.01 0.01 0.01; visual box size=0.01 0.01 0.01
- link IR7: geometry collision box size=0.01 0.01 0.01; visual box size=0.01 0.01 0.01
- link base_link: geometry collision cylinder length=0.07 radius=0.07; visual cylinder length=0.08 radius=0.07
- link left_wheel: geometry collision cylinder length=0.007 radius=0.04; visual cylinder length=0.007 radius=0.04
- link right_wheel: geometry collision cylinder length=0.007 radius=0.04; visual cylinder length=0.007 radius=0.04
Joints:
- removed joint base_to_arrow
- removed joint base_to_cam
- removed joint base_to_led0
- removed joint base_to_led1
- removed joint base_to_led2
- removed joint base_to_led3
- removed joint base_to_led4
- removed joint base_to_led5
- removed joint base_to_led6
- removed joint base_to_led7
- removed joint base_to_top
- joint base_to_IR0: origin xyz=0.155 -0.041 0.125 rpy=1.57 0 1.30890 -> xyz= 0.06975, -0.01845 0.1 rpy=1.57 0 1.27
- joint base_to_IR1: origin xyz=0.113 -0.113 0.125 rpy=1.57 0 0.78530 -> xyz=0.05085 -0.05085 0.1 rpy=1.57 0 0.77
- joint base_to_IR2: origin xyz=0.0 -0.16 0.125 rpy=1.57 0 6.2830 -> xyz=0.0 -0.072 0.1 rpy=1.57 0 0
- joint base_to_IR3: origin xyz=-0.139 -0.08 0.125 rpy=1.57 0 5.23589 -> xyz=-0.06255, -0.036 0.1 rpy=1.57 0 5.21
- joint base_to_IR4: origin xyz=-0.139 0.08 0.125 rpy=1.57 0 4.1886 -> xyz=-0.06255, 0.036 0.1 rpy=1.57 0 4.21
- joint base_to_IR5: origin xyz=0.0 0.16 0.125 rpy=1.57 0 3.1415 -> xyz=0.0 0.072 0.1 rpy=1.57 0 3.1415
- joint base_to_IR6: origin xyz=0.113 0.113 0.125 rpy=1.57 0 2.356 -> xyz=0.05085 0.05085 0.1 rpy=1.57 0 2.37
- joint base_to_IR7: origin xyz=0.155 0.041 0.125 rpy=1.57 0 1.8324 -> xyz=0.06975 0.01845  0.1 rpy=1.57 0 1.87
- joint base_to_left_wheel: child left_wheel -> right_wheel; origin xyz=0.007 0.12 0.078 rpy=0 0 0 -> xyz=0 0.078 0.043 rpy=0 0 0
- joint base_to_right_wheel: child right_wheel -> left_wheel; origin xyz=0.007 -0.12 0.078 rpy=0 0 0 -> xyz=0 -0.078 0.043 rpy=0 0 0
