Commit message: FlatWorld class added. Bug detected (working on it): variability of results in different computers. Robot scaled x2.

File: mereli/models/entities/wall/wall.urdf (robot description, URDF)
Before this commit: robot wall, 1 links, 0 joints
Links:
- link baseLink: mass 0 -> 10

File: mereli/models/tmp/wall_1x101x1.urdf (robot description, URDF)
Before this commit: robot wall, 1 links, 0 joints
Links:
- link baseLink: mass 0 -> 10; geometry collision box size=1 101 1; visual box size=1 101 1

File: mereli/models/tmp/wall_1x11x1.urdf (robot description, URDF)
Before this commit: robot wall, 1 links, 0 joints
Links:
- link baseLink: mass 0 -> 1000; geometry collision box size=1 11 1; visual box size=1 11 1

File: mereli/models/tmp/wall_1x6x1.urdf (robot description, URDF)
Before this commit: robot wall, 1 links, 0 joints
Links:
- link baseLink: mass 0 -> 1000

File: mereli/models/tmp/wall_4x1x1.urdf (robot description, URDF)
Before this commit: robot wall, 1 links, 0 joints
Links:
- link baseLink: mass 0 -> 1000

File: mereli/models/tmp/wall_99x1x1.urdf (robot description, URDF)
Before this commit: robot wall, 1 links, 0 joints
Links:
- link baseLink: mass 0 -> 10; geometry collision box size=99 1 1; visual box size=99 1 1

File: mereli/models/tmp/wall_9x1x1.urdf (robot description, URDF)
Before this commit: robot wall, 1 links, 0 joints
Links:
- link baseLink: mass 1000.0 -> 1000; geometry collision box size=9 1 1; visual box size=9 1 1
