Commit message: Fixed wall dimensions. Some modif. in basic example 2.

File: mereli/models/tmp/wall_0.1x3.1x0.1.urdf (robot description, URDF)
Before this commit: robot wall, 1 links, 0 joints
Links:
- link baseLink: mass 1000 -> 10; geometry collision box size=0.1 3.1 0.1; visual box size=0.1 3.1 0.1

File: mereli/models/tmp/wall_0.1x3.1x0.2.urdf (robot description, URDF)
Before this commit: robot wall, 1 links, 0 joints
Links:
- link baseLink: mass 1000 -> 10; geometry collision box size=0.1 3.1 0.2; visual box size=0.1 3.1 0.2

File: mereli/models/tmp/wall_2.9x0.1x0.1.urdf (robot description, URDF)
Before this commit: robot wall, 1 links, 0 joints
Links:
- link baseLink: geometry collision box size=2.9 0.1 0.1; visual box size=2.9 0.1 0.1

File: mereli/models/tmp/wall_2.9x0.1x0.2.urdf (robot description, URDF)
Before this commit: robot wall, 1 links, 0 joints
Links:
- link baseLink: mass 1000 -> 10; geometry collision box size=2.9 0.1 0.2; visual box size=2.9 0.1 0.2
