Commit message: Minor changes .

File: mereli/models/tmp/wall_0.1x20.1x1.urdf (robot description, URDF)
Before this commit: robot wall, 1 links, 0 joints
Links:
- link baseLink: geometry collision box size=0.1 20.1 1; visual box size=0.1 20.1 1

File: mereli/models/tmp/wall_0.1x3.1x0.2.urdf (robot description, URDF)
Before this commit: robot wall, 1 links, 0 joints
Links:
- link baseLink: geometry collision box size=0.1 3.1 0.2; visual box size=0.1 3.1 0.2

File: mereli/models/tmp/wall_0.1x4.1x0.2.urdf (robot description, URDF)
Before this commit: robot wall, 1 links, 0 joints
Links:
- link baseLink: geometry collision box size=0.1 4.1 0.2; visual box size=0.1 4.1 0.2

File: mereli/models/tmp/wall_1.9x0.05x1.urdf (robot description, URDF)
Before this commit: robot wall, 1 links, 0 joints
Links:
- link baseLink: geometry collision box size=1.9 0.05 1; visual box size=1.9 0.05 1

File: mereli/models/tmp/wall_19.9x0.1x1.urdf (robot description, URDF)
Before this commit: robot wall, 1 links, 0 joints
Links:
- link baseLink: geometry collision box size=19.9 0.1 1; visual box size=19.9 0.1 1

File: mereli/models/tmp/wall_2.9x0.1x0.2.urdf (robot description, URDF)
Before this commit: robot wall, 1 links, 0 joints
Links:
- link baseLink: geometry collision box size=2.9 0.1 0.2; visual box size=2.9 0.1 0.2

File: mereli/models/tmp/wall_3.9x0.1x0.2.urdf (robot description, URDF)
Before this commit: robot wall, 1 links, 0 joints
Links:
- link baseLink: geometry collision box size=3.9 0.1 0.2; visual box size=3.9 0.1 0.2
