Commit message: Minor modif.

File: mereli/models/maps/simple_map_2/simple_map_2.urdf (robot description, URDF)
Before this commit: robot simple_map_2, 1 links, 0 joints
Links:
- link baseLink: geometry collision mesh filename=simple_map_2.obj scale=0.4 0.4 0.4; visual mesh filename=simple_map_2.obj scale=0.4 0.4 0.4

Commit message: Experiment modifications.

File: mereli/models/maps/simple_map_2/simple_map_2.urdf (robot description, URDF)
Before this commit: robot simple_map_2, 1 links, 0 joints
Links:
- link baseLink: geometry collision mesh filename=simple_map_2.obj scale=1 1 1; visual mesh filename=simple_map_2.obj scale=1 1 1

File: mereli/models/tmp/wall_0.5x3.5x1.urdf (robot description, URDF)
Before this commit: robot wall, 1 links, 0 joints
Links:
- link baseLink: geometry collision box size=0.5 3.5 1; visual box size=0.5 3.5 1

File: mereli/models/tmp/wall_1x11x1.urdf (robot description, URDF)
Before this commit: robot wall, 1 links, 0 joints
Links:
- link baseLink: mass 10 -> 1000; geometry collision box size=1 11 1; visual box size=1 11 1

File: mereli/models/tmp/wall_4x1x1.urdf (robot description, URDF)
Before this commit: robot wall, 1 links, 0 joints
Links:
- link baseLink: mass 10 -> 1000; geometry collision box size=4 1 1; visual box size=4 1 1

File: mereli/models/tmp/wall_9x1x1.urdf (robot description, URDF)
Before this commit: robot wall, 1 links, 0 joints
Links:
- link baseLink: mass 10 -> 1000; geometry collision box size=9 1 1; visual box size=9 1 1
