Commit message: Huge commit: IRIN examples, IRIN sensors, New sensor reading, new actuator planning, Comm Space foraging, comm space perforance increase,etc

File: mereli/models/entities/ball/ball.urdf (robot description, URDF)
Before this commit: robot light, 1 links, 0 joints
Links:
- removed link baseLink
- added link base_link, mass 10; collision sphere radius=1

File: mereli/models/entities/epuck/epuck.urdf.xacro (robot description, xacro)
@@ -583,4 +583,46 @@
             <origin xyz="0 0 0" rpy="0 0 6.0213"/>
             <ghost link='ghost_cone_DS7'/>
+        </sector>
+    </sensor>
+    <sensor name="light_sensor">
+       <sector index="0">
+            <parent link="IR0"/>
+            <origin xyz="0 0 0" rpy="0 0 0.26179"/>
+            <ghost link='ghost_cone_LS0'/>
+        </sector>
+        <sector index="1">
+            <parent link="IR1"/>
+            <origin xyz="0 0 0" rpy="0 0 0.78539"/>
+            <ghost link='ghost_cone_LS1'/>
+        </sector>
+        <sector index="2">
+            <parent link="IR2"/>
+            <origin xyz="0 0 0" rpy="0 0 1.57079"/>
+            <ghost link='ghost_cone_LS2'/>
+        </sector>
+        <sector index="3">
+            <parent link="IR3"/>
+            <origin xyz="0 0 0" rpy="0 0 2.61799"/>
+            <ghost link='ghost_cone_LS3'/>
+        </sector>
+        <sector index="4">
+            <parent link="IR4"/>
+            <origin xyz="0 0 0" rpy="0 0 3.66519"/>
+            <ghost link='ghost_cone_LS4'/>
+        </sector>
+        <sector index="5">
+            <parent link="IR5"/>
+            <origin xyz="0 0 0" rpy="0 0 4.71238"/>
+            <ghost link='ghost_cone_LS5'/>
+        </sector>
+        <sector index="6">
+            <parent link="IR6"/>
+            <origin xyz="0 0 0" rpy="0 0 5.49778"/>
+            <ghost link='ghost_cone_LS6'/>
+        </sector>
+        <sector index="7">
+            <parent link="IR7"/>
+            <origin xyz="0 0 0" rpy="0 0 6.0213"/>
+            <ghost link='ghost_cone_LS7'/>
         </sector>
     </sensor>
@@ -724,13 +766,13 @@
       <origin rpy="0 0 0" xyz="0 0 0"/>
       <geometry>
-			 <mesh filename="ghost_DS.obj" scale="0.5 0.5 0.5"/>
+			 <mesh filename="ghost_DS.obj" scale="1 2 1"/>
       </geometry>
       <material name="transparent_red">
-        <color rgba="1 0 0 0.0"/>
+        <color rgba="1 0 0 0.7"/>
       </material>
     </visual>
      <collision>
             <geometry>
-            <mesh filename="ghost_DS.obj" scale="0.5 0.5 0.5"/>
+            <mesh filename="ghost_DS.obj" scale="1 2 1"/>
             </geometry>
             <origin xyz="0 0 0" />
@@ -751,5 +793,5 @@
       <origin rpy="0 0 0" xyz="0 0 0.0"/>
       <geometry>
-			 <mesh filename="ghost_DS.obj" scale="0.5 0.5 0.5"/>
+            <mesh filename="ghost_DS.obj" scale="1 2 1"/>
       </geometry>
       <material name="transparent_red">
@@ -759,5 +801,5 @@
     <collision>
             <geometry>
-            <mesh filename="ghost_DS.obj" scale="0.5 0.5 0.5"/>
+            <mesh filename="ghost_DS.obj" scale="1 2 1"/>
             </geometry>
             <origin xyz="0 0 0" />
@@ -778,5 +820,5 @@
       <origin rpy="0 0 0" xyz="0 0 0.0"/>
       <geometry>
-			 <mesh filename="ghost_DS.obj" scale="0.5 0.5 0.5"/>
+			 <mesh filename="ghost_DS.obj" scale="1 2 1"/>
       </geometry>
       <material name="transparent_red">
@@ -786,5 +828,5 @@
          <collision>
             <geometry>
-            <mesh filename="ghost_DS.obj" scale="0.5 0.5 0.5"/>
+			 <mesh filename="ghost_DS.obj" scale="1 2 1"/>
             </geometry>
             <origin xyz="0 0 0" />
@@ -805,5 +847,5 @@
       <origin rpy="0 0 0" xyz="0 0 0.0"/>
       <geometry>
-			 <mesh filename="ghost_DS.obj" scale="0.5 0.5 0.5"/>
+            <mesh filename="ghost_DS.obj" scale="1 2 1"/>
       </geometry>
       <material name="transparent_red">
@@ -813,5 +855,5 @@
          <collision>
             <geometry>
-            <mesh filename="ghost_DS.obj" scale="0.5 0.5 0.5"/>
+            <mesh filename="ghost_DS.obj" scale="1 2 1"/>
             </geometry>
             <origin xyz="0 0 0" />
@@ -832,5 +874,5 @@
       <origin rpy="0 0 0" xyz="0 0 0"/>
       <geometry>
-			 <mesh filename="ghost_DS.obj" scale=".5 .5 .5"/>
+            <mesh filename="ghost_DS.obj" scale="1 2 1"/>
       </geometry>
       <material name="transparent_red">
@@ -840,5 +882,5 @@
          <collision>
             <geometry>
-            <mesh filename="ghost_DS.obj" scale=".5 .5 .5"/>
+            <mesh filename="ghost_DS.obj" scale="1 2 1"/>
             </geometry>
             <origin xyz="0 0 0" />
@@ -859,5 +901,5 @@
       <origin rpy="0 0 0" xyz="0 0 0"/>
       <geometry>
-			 <mesh filename="ghost_DS.obj" scale=".5 .5 .5"/>
+            <mesh filename="ghost_DS.obj" scale="1 2 1"/>
       </geometry>
       <material name="transparent_red">
@@ -886,5 +928,5 @@
       <origin rpy="0 0 0" xyz="0 0 0"/>
       <geometry>
-			 <mesh filename="ghost_DS.obj" scale=".5 .5 .5"/>
+            <mesh filename="ghost_DS.obj" scale="1 2 1"/>
       </geometry>
       <material name="transparent_red">
@@ -894,5 +936,5 @@
          <collision>
             <geometry>
-            <mesh filename="ghost_DS.obj" scale=".5 .5 .5"/>
+            <mesh filename="ghost_DS.obj" scale="1 2 1"/>
             </geometry>
             <origin xyz="0 0 0" />
@@ -913,5 +955,5 @@
         <origin rpy="0 0 0" xyz="0 0 0"/>
         <geometry>
-                <mesh filename="ghost_DS.obj" scale=".5 .5 ..5"/>
+            <mesh filename="ghost_DS.obj" scale="1 2 1"/>
         </geometry>
         <material name="transparent_red">
@@ -921,5 +963,5 @@
             <collision>
                 <geometry>
-                <mesh filename="ghost_DS.obj" scale=".5 .5 .5"/>
+            <mesh filename="ghost_DS.obj" scale="1 2 1"/>
                 </geometry>
                 <origin xyz="0 0 0" />
